Commit message: urdf directory added

File: plz_plz_description/urdf/plz_plz.xacro (robot description, xacro)
@@ -4,4 +4,9 @@
 <xacro:include filename="$(find plz_plz_description)/urdf/plz_plz.trans" />
 <xacro:include filename="$(find plz_plz_description)/urdf/plz_plz.gazebo" />
+<link name="world" />
+<joint name="Dummy" type="fixed">
+  <parent link="world"/>
+  <child link="base_link"/>
+</joint>
 <link name="base_link">
   <inertial>
@@ -470,5 +475,5 @@
   <child link="alternate_design_top_1"/>
 </joint>
-<joint name="joint_1" type="continuous">
+<joint name="Rev6" type="continuous">
   <origin rpy="0 0 0" xyz="0.136 -0.092 0.1555"/>
   <parent link="combined_servo_2_1"/>
@@ -481,5 +486,5 @@
   <child link="combined_servo_v1_1"/>
 </joint>
-<joint name="joint_2" type="continuous">
+<joint name="Rev8" type="continuous">
   <origin rpy="0 0 0" xyz="0.0 0.0 0.0"/>
   <parent link="combined_servo_v1_1"/>
@@ -487,5 +492,5 @@
   <axis xyz="-0.0 1.0 0.0"/>
 </joint>
-<joint name="joint_3" type="continuous">
+<joint name="Rev9" type="continuous">
   <origin rpy="0 0 0" xyz="0.11 0.0 0.0"/>
   <parent link="link_2_drive_side_1_1"/>
@@ -508,5 +513,5 @@
   <child link="combined_servo_444_1"/>
 </joint>
-<joint name="joint_4" type="continuous">
+<joint name="Rev13" type="continuous">
   <origin rpy="0 0 0" xyz="0.0 0.0 -0.04"/>
   <parent link="combined_servo_444_1"/>
